File: 14_pin_pmt_Rev2.kicad_sch (KiCad schematic)
At the start: 41 parts, among them J1 Dynode 1, J10 Dynode 10, J11 Anode, J12 Pin1, J13 Focus, J14 Cathode, J15 Signal, J17 GND, J2 Dynode 2, J3 Dynode 3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

Commit message: added title blocks
Other:
- company: (none) -> Gigstorm
- title: (none) -> 14 Pin PMT Voltage Divider
Changed lines of the file:
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@@
 (kicad_sch (version 20230121) (generator eeschema)
   (paper "A4")
+  (title_block
+    (title "14 Pin PMT Voltage Divider")
+    (date "2023-08-03")
+    (rev "2.0")
+    (company "Gigstorm")
+  )
   (junction (at 116.84 73.66) (diameter 0) (color 0 0 0 0)
   )
